File: Hardware/Schematics/System interconnections.kicad_sch (KiCad schematic)
At the start: 10 parts, among them Q1 2N2222, Q2 D1207

Commit message: Reupload schematics
Connections:
- net at LM393. (VCC): now also ESP32. (3.3V)
- net at ESP32. (3.3V): no longer LM393. (VCC)
- new net: ESP32. (3.3V), LM393. (VCC) (x2)
- now unconnected: ESP32. (3.3V), ESP32. (3.3V)
